Commit message: Update: task2_with_arm

File: src/robot_arm_v2/urdf/robot_arm_v2.urdf (robot description, URDF)
Before this commit: robot None, 7 links, 6 joints
Joints:
- joint gripper_base_left_joint: limit lower=-1.18 upper=0 effort=300 velocity=2 -> lower=-1.57 upper=1.57 effort=300 velocity=2

Commit message: Tuning

File: src/robot_arm_v2/urdf/robot_arm_v2.urdf (robot description, URDF)
Before this commit: robot None, 7 links, 6 joints
Joints:
- joint arm1_arm2_joint: axis 0 -1 0 -> 0 1 0
