Commit message: Tuning

File: src/robot_arm_v2/urdf/robot_arm_v2.ros2_control.xacro (robot description, xacro)
@@ -1,49 +1,40 @@
 <?xml version="1.0"?>
 <robot xmlns:xacro="http://www.ros.org/wiki/xacro">
-        <ros2_control name="Arm" type="system">
-            <hardware>
-            <!-- <plugin>arduino_arm_hardware::ArduinoArmHardwareInterface</plugin>
-                <param name="port">/dev/ttyACM0</param> -->
-                <!-- <plugin>mock_components/GenericSystem</plugin> -->
+    <ros2_control name="ArmWithGripper" type="system">
+        <hardware>
             <plugin>rpi_arm_hardware::RPiArmHardwareInterface</plugin>
-                <param name="host">127.0.0.1</param>
-                <param name="port">9999</param>
-            </hardware>
-            <joint name="base_rotating_waste_joint">
-                <command_interface name="position"/>
-                <state_interface name="position">
-                  <param name="initial_value">0.0</param>
-                </state_interface>
-            </joint>
-            <joint name="rotating_waste_arm1_joint">
-                <command_interface name="position"/>
-                <state_interface name="position">
-                  <param name="initial_value">0.0</param>
-                </state_interface>
-            </joint>
-            <joint name="arm1_arm2_joint">
-                <command_interface name="position"/>
-                <state_interface name="position">
-                  <param name="initial_value">0.0</param>
-                </state_interface>
-            </joint>
-            <joint name="arm2_gripper_base_joint">
-                <command_interface name="position"/>
-                <state_interface name="position">
-                  <param name="initial_value">0.0</param>
-                </state_interface>
-            </joint>
-        </ros2_control>
-        <!-- Gripper system -->
-        <ros2_control name="Gripper" type="system">
-            <hardware>
-                <plugin>mock_components/GenericSystem</plugin>
-            </hardware>
-            <joint name="gripper_base_left_joint">
-                <command_interface name="position"/>
-                <state_interface name="position">
-                  <param name="initial_value">0.0</param>
-                </state_interface>
-            </joint>
-        </ros2_control>
+            <param name="host">127.0.0.1</param>
+            <param name="port">9999</param>
+        </hardware>
+        <joint name="base_rotating_waste_joint">
+            <command_interface name="position"/>
+            <state_interface name="position">
+                <param name="initial_value">0.0</param>
+            </state_interface>
+        </joint>
+        <joint name="rotating_waste_arm1_joint">
+            <command_interface name="position"/>
+            <state_interface name="position">
+                <param name="initial_value">0.0</param>
+            </state_interface>
+        </joint>
+        <joint name="arm1_arm2_joint">
+            <command_interface name="position"/>
+            <state_interface name="position">
+                <param name="initial_value">0.0</param>
+            </state_interface>
+        </joint>
+        <joint name="arm2_gripper_base_joint">
+            <command_interface name="position"/>
+            <state_interface name="position">
+                <param name="initial_value">0.0</param>
+            </state_interface>
+        </joint>
+        <joint name="gripper_base_left_joint">
+            <command_interface name="position"/>
+            <state_interface name="position">
+                <param name="initial_value">0.0</param>
+            </state_interface>
+        </joint>
+    </ros2_control>
 </robot>

File: src/robot_arm_v2/urdf/robot_arm_v2.urdf (robot description, URDF)
Before this commit: robot None, 7 links, 6 joints
Joints:
- joint arm1_arm2_joint: limit lower=-0.972 upper=2.172 effort=300 velocity=2 -> lower=-2.35 upper=0.78 effort=300 velocity=2
